File: Hardware/MegaMouse/mcu.kicad_sch (KiCad schematic)
At the start: 18 parts, among them J401 ICSP, SW401 RESET, SW402 START_SW, SW403 STOP/MODE_SW, U401 ATmega328P, Y401 16mHz

Commit message: Even more stuff! also bump libs
Changed lines of the file:
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@@
     (stroke (width 0) (type default) (color 0 0 0 0))
   )
-  (wire (pts (xy 57.785 61.595) (xy 81.28 61.595))
+  (wire (pts (xy 57.785 61.595) (xy 79.375 61.595))
     (stroke (width 0) (type default) (color 0 0 0 0))
   )
@@
     (stroke (width 0) (type default) (color 0 0 0 0))
   )
+  (wire (pts (xy 57.785 59.055) (xy 79.375 59.055))
+    (stroke (width 0) (type default) (color 0 0 0 0))
+  )
   (wire (pts (xy 100.33 94.615) (xy 106.68 94.615))
     (stroke (width 0) (type default) (color 0 0 0 0))
@@
     (stroke (width 0) (type default) (color 0 0 0 0))
   )
-  (wire (pts (xy 57.785 56.515) (xy 81.28 56.515))
-    (stroke (width 0) (type default) (color 0 0 0 0))
-  )
-  (wire (pts (xy 57.785 59.055) (xy 81.28 59.055))
+  (wire (pts (xy 57.785 56.515) (xy 79.375 56.515))
     (stroke (width 0) (type default) (color 0 0 0 0))
   )
@@
     (effects (font (size 1.27 1.27)) (justify right bottom))
   )
-  (label "SDI" (at 78.74 59.055 180)
+  (label "SDI" (at 79.375 59.055 180)
     (effects (font (size 1.27 1.27)) (justify right bottom))
   )
@@
     (effects (font (size 1.27 1.27)) (justify right))
   )
-  (hierarchical_label "SDI" (shape input) (at 81.28 59.055 0)
-    (effects (font (size 1.27 1.27)) (justify left))
-  )
-  (hierarchical_label "SDO" (shape output) (at 81.28 56.515 0)
-    (effects (font (size 1.27 1.27)) (justify left))
-  )
   (hierarchical_label "RXD" (shape input) (at 106.68 92.075 0)
     (effects (font (size 1.27 1.27)) (justify left))
   )
-  (hierarchical_label "SCK" (shape output) (at 81.28 61.595 0)
-    (effects (font (size 1.27 1.27)) (justify left))
-  )

Commit message: Bump config
Other:
- company: SNHU -> Kitsune Scientific
- title: Inverted Pendulum Controller -> MegaMouse
Changed lines of the file:
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@@
   (paper "A4")
   (title_block
-    (title "Inverted Pendulum Controller")
+    (title "MegaMouse")
     (date "${ISSUE}")
     (rev "${REVISION}")
-    (company "SNHU")
+    (company "Kitsune Scientific")
     (comment 4 "Release: ${FULL_REVISION}")
   )
