File: Hardware/MegaMouse/mcu.kicad_sch (KiCad schematic)
At the start: 18 parts, among them J401 ICSP, SW401 RESET, SW402 START_SW, SW403 STOP/MODE_SW, U401 ATmega328P, Y401 16mHz

Commit message: Awesomeness
Parts:
- removed R406: 10K, Resistor_SMD:R_0805_2012Metric, symbol Device:R_Small
- removed SW403: STOP/MODE_SW, Button_Switch_THT:SW_PUSH_6mm_H5mm, symbol Switch:SW_Push
- C403, C404: footprint Capacitor_SMD:C_0805_2012Metric -> Capacitor_SMD:C_0201_0603Metric
- SW402: value START_SW -> START/MODE; footprint Button_Switch_THT:SW_PUSH_6mm_H5mm -> Button_Switch_THT:SW_Tactile_SKHH_Angled
Connections:
- net STOP/MODE is gone; now on net START/MODE: U401.12 (PB0)
- net LATCH_OUT: now reaches U401.14 (PB2)
- net CLOCK_OUT: now reaches U401.32 (PD2)
- net START renamed START/MODE
- net START/MODE: no longer U401.13 (PB1)
- new net DATA_OUT: U401.13 (PB1)
Other:
- moved on the sheet: D401, R403

Commit message: Add decoupling caps and 3d models
Parts:
- added C402: 100nF, Capacitor_SMD:C_0805_2012Metric, symbol Device:C_Small
- renumbered C402 to C403, C403 to C404, C404 to C405
Connections:
- net +5V: now also C402.1
- net GND: now also C402.2
Changed lines of the file:
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@@
+    (stroke (width 0) (type default) (color 0 0 0 0))
+  )
+  (wire (pts (xy 27.94 35.56) (xy 27.94 36.83))
     (stroke (width 0) (type default) (color 0 0 0 0))
   )
@@
   )
   (wire (pts (xy 24.13 157.48) (xy 35.56 157.48))
+    (stroke (width 0) (type default) (color 0 0 0 0))
+  )
+  (wire (pts (xy 27.94 29.21) (xy 27.94 30.48))
     (stroke (width 0) (type default) (color 0 0 0 0))
   )
@@
   (symbol (lib_name "GND_8") (lib_id "power:GND") (at 42.545 120.015 0) (unit 1)
     (in_bom yes) (on_board yes)
-    (property "Reference" "#PWR0404" (id 0) (at 42.545 126.365 0)
+    (property "Reference" "#PWR0406" (id 0) (at 42.545 126.365 0)
       (effects (font (size 1.27 1.27)) hide)
     )
@@
     (pin "2")
   )
+  (symbol (lib_id "Device:C_Small") (at 27.94 33.02 0) (unit 1)
+    (in_bom yes) (on_board yes)
+    (property "Reference" "C402" (id 0) (at 20.32 31.75 0)
+      (effects (font (size 1.27 1.27)) (justify left))
+    )
+    (property "Value" "100nF" (id 1) (at 20.32 34.29 0)
+      (effects (font (size 1.27 1.27)) (justify left))
+    )
+    (property "Footprint" "Capacitor_SMD:C_0805_2012Metric" (id 2) (at 27.94 33.02 0)
+      (effects (font (size 1.27 1.27)) hide)
+    )
+    (property "Datasheet" "~" (id 3) (at 27.94 33.02 0)
+      (effects (font (size 1.27 1.27)) hide)
+    )
+    (pin "1")
+    (pin "2")
+  )
   (symbol (lib_name "GND_9") (lib_id "power:GND") (at 85.09 79.375 0) (unit 1)
     (in_bom yes) (on_board yes)
-    (property "Reference" "#PWR0408" (id 0) (at 85.09 85.725 0)
+    (property "Reference" "#PWR0410" (id 0) (at 85.09 85.725 0)
       (effects (font (size 1.27 1.27)) hide)
     )
@@
   (symbol (lib_name "+5V_6") (lib_id "power:+5V") (at 50.165 148.59 0) (unit 1)
     (in_bom yes) (on_board yes)
-    (property "Reference" "#PWR0406" (id 0) (at 50.165 152.4 0)
+    (property "Reference" "#PWR0408" (id 0) (at 50.165 152.4 0)
       (effects (font (size 1.27 1.27)) hide)
     )
@@
   (symbol (lib_name "GND_5") (lib_id "power:GND") (at 50.165 161.925 0) (unit 1)
     (in_bom yes) (on_board yes)
-    (property "Reference" "#PWR0407" (id 0) (at 50.165 168.275 0)
+    (property "Reference" "#PWR0409" (id 0) (at 50.165 168.275 0)
       (effects (font (size 1.27 1.27)) hide)
     )
@@
   (symbol (lib_name "+5V_7") (lib_id "power:+5V") (at 38.1 29.21 0) (unit 1)
     (in_bom yes) (on_board yes)
-    (property "Reference" "#PWR0402" (id 0) (at 38.1 33.02 0)
+    (property "Reference" "#PWR0404" (id 0) (at 38.1 33.02 0)
       (effects (font (size 1.27 1.27)) hide)
     )
@@
   (symbol (lib_id "Device:C_Small") (at 38.1 33.02 0) (unit 1)
     (in_bom yes) (on_board yes)
-    (property "Reference" "C402" (id 0) (at 30.48 31.75 0)
+    (property "Reference" "C403" (id 0) (at 30.48 31.75 0)
       (effects (font (size 1.27 1.27)) (justify left))
     )
@@
   (symbol (lib_id "Device:C_Small") (at 89.535 74.295 0) (unit 1)
     (in_bom yes) (on_board yes)
-    (property "Reference" "C404" (id 0) (at 92.075 74.295 0)
+    (property "Reference" "C405" (id 0) (at 92.075 74.295 0)
       (effects (font (size 1.27 1.27)) (justify left))
     )
@@
   (symbol (lib_name "GND_4") (lib_id "power:GND") (at 146.05 33.655 0) (unit 1)
     (in_bom yes) (on_board yes)
-    (property "Reference" "#PWR0411" (id 0) (at 146.05 40.005 0)
+    (property "Reference" "#PWR0413" (id 0) (at 146.05 40.005 0)
       (effects (font (size 1.27 1.27)) hide)
     )
@@
   (symbol (lib_name "+5V_5") (lib_id "power:+5V") (at 130.81 23.495 0) (unit 1)
     (in_bom yes) (on_board yes)
-    (property "Reference" "#PWR0410" (id 0) (at 130.81 27.305 0)
+    (property "Reference" "#PWR0412" (id 0) (at 130.81 27.305 0)
       (effects (font (size 1.27 1.27)) hide)
     )
@@
   (symbol (lib_name "+5V_3") (lib_id "power:+5V") (at 187.96 24.765 0) (unit 1)
     (in_bom yes) (on_board yes)
-    (property "Reference" "#PWR0414" (id 0) (at 187.96 28.575 0)
+    (property "Reference" "#PWR0415" (id 0) (at 187.96 28.575 0)
       (effects (font (size 1.27 1.27)) hide)
     )
@@
   (symbol (lib_id "Device:C_Small") (at 80.645 74.295 0) (unit 1)
     (in_bom yes) (on_board yes)
-    (property "Reference" "C403" (id 0) (at 73.025 74.295 0)
+    (property "Reference" "C404" (id 0) (at 73.025 74.295 0)
       (effects (font (size 1.27 1.27)) (justify left))
     )
@@
     (pin "1")
     (pin "2")
+  )
+  (symbol (lib_name "+5V_7") (lib_id "power:+5V") (at 27.94 29.21 0) (unit 1)
+    (in_bom yes) (on_board yes)
+    (property "Reference" "#PWR0402" (id 0) (at 27.94 33.02 0)
+      (effects (font (size 1.27 1.27)) hide)
+    )
+    (property "Value" "+5V" (id 1) (at 27.94 25.4 0))
+    (property "Footprint" "" (id 2) (at 27.94 29.21 0)
+      (effects (font (size 1.27 1.27)) hide)
+    )
+    (property "Datasheet" "" (id 3) (at 27.94 29.21 0)
+      (effects (font (size 1.27 1.27)) hide)
+    )
+    (pin "1")
   )
   (symbol (lib_id "Switch:SW_Push") (at 139.7 32.385 0) (unit 1)
@@
     (pin "1")
   )
+  (symbol (lib_name "GND_7") (lib_id "power:GND") (at 27.94 36.83 0) (unit 1)
+    (in_bom yes) (on_board yes)
+    (property "Reference" "#PWR0403" (id 0) (at 27.94 43.18 0)
+      (effects (font (size 1.27 1.27)) hide)
+    )
+    (property "Value" "GND" (id 1) (at 27.94 40.64 0))
+    (property "Footprint" "" (id 2) (at 27.94 36.83 0)
+      (effects (font (size 1.27 1.27)) hide)
+    )
+    (property "Datasheet" "" (id 3) (at 27.94 36.83 0)
+      (effects (font (size 1.27 1.27)) hide)
+    )
+    (pin "1")
+  )
   (symbol (lib_id "Switch:SW_Push") (at 180.34 27.305 0) (unit 1)
     (in_bom yes) (on_board yes)
@@
   (symbol (lib_name "GND_10") (lib_id "power:GND") (at 113.665 24.13 0) (unit 1)
     (in_bom yes) (on_board yes)
-    (property "Reference" "#PWR0409" (id 0) (at 113.665 30.48 0)
+    (property "Reference" "#PWR0411" (id 0) (at 113.665 30.48 0)
       (effects (font (size 1.27 1.27)) hide)
     )
@@
   (symbol (lib_name "GND_3") (lib_id "power:GND") (at 173.355 36.195 0) (unit 1)
     (in_bom yes) (on_board yes)
-    (property "Reference" "#PWR0412" (id 0) (at 173.355 42.545 0)
+    (property "Reference" "#PWR0414" (id 0) (at 173.355 42.545 0)
       (effects (font (size 1.27 1.27)) hide)
     )
@@
   (symbol (lib_name "+5V_8") (lib_id "power:+5V") (at 43.815 37.465 0) (unit 1)
     (in_bom yes) (on_board yes)
-    (property "Reference" "#PWR0405" (id 0) (at 43.815 41.275 0)
+    (property "Reference" "#PWR0407" (id 0) (at 43.815 41.275 0)
       (effects (font (size 1.27 1.27)) hide)
     )
@@
   (symbol (lib_name "GND_7") (lib_id "power:GND") (at 38.1 36.83 0) (unit 1)
     (in_bom yes) (on_board yes)
-    (property "Reference" "#PWR0403" (id 0) (at 38.1 43.18 0)
-      (effects (font (size 1.27 1.27)) hide)
-    )
+    (property "Reference" "#PWR0405" (id 0) (at 38.1 43.18 0)
+      (effects (font (size 1.27 1.27)) hide)
+    )

Commit message: Fix crystal
Parts:
- C404, C405: footprint Capacitor_SMD:C_0201_0603Metric -> Capacitor_SMD:C_0603_1608Metric
Changed lines of the file:
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@@
       (effects (font (size 1.27 1.27)) (justify left))
     )
-    (property "Footprint" "Capacitor_SMD:C_0201_0603Metric" (id 2) (at 89.535 74.295 0)
+    (property "Footprint" "Capacitor_SMD:C_0603_1608Metric" (id 2) (at 89.535 74.295 0)
       (effects (font (size 1.27 1.27)) hide)
     )
@@
       (effects (font (size 1.27 1.27)) (justify left))
     )
-    (property "Footprint" "Capacitor_SMD:C_0201_0603Metric" (id 2) (at 80.645 74.295 0)
+    (property "Footprint" "Capacitor_SMD:C_0603_1608Metric" (id 2) (at 80.645 74.295 0)
       (effects (font (size 1.27 1.27)) hide)
     )

Commit message: Add more wiring
Parts:
- added TP401, TP402, TP403, TP404: TestPoint, TestPoint:TestPoint_Pad_2.0x2.0mm, symbol Connector:TestPoint
Connections:
- net RST: now also TP404.1
- net SCK: now also TP402.1
- net SDI: now also TP403.1
- net SDO: now also TP401.1
Changed lines of the file:
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@@
+    (stroke (width 0) (type default) (color 0 0 0 0))
+  )
+  (wire (pts (xy 69.85 144.145) (xy 74.93 144.145))
     (stroke (width 0) (type default) (color 0 0 0 0))
   )
@@
     (stroke (width 0) (type default) (color 0 0 0 0))
   )
+  (wire (pts (xy 69.85 154.305) (xy 74.93 154.305))
+    (stroke (width 0) (type default) (color 0 0 0 0))
+  )
   (wire (pts (xy 24.13 160.02) (xy 35.56 160.02))
     (stroke (width 0) (type default) (color 0 0 0 0))
@@
     (stroke (width 0) (type default) (color 0 0 0 0))
   )
+  (wire (pts (xy 69.85 149.225) (xy 74.93 149.225))
+    (stroke (width 0) (type default) (color 0 0 0 0))
+  )
   (wire (pts (xy 57.785 66.675) (xy 80.645 66.675))
     (stroke (width 0) (type default) (color 0 0 0 0))
@@
   )
   (wire (pts (xy 85.09 78.74) (xy 89.535 78.74))
+    (stroke (width 0) (type default) (color 0 0 0 0))
+  )
+  (wire (pts (xy 69.85 159.385) (xy 74.93 159.385))
     (stroke (width 0) (type default) (color 0 0 0 0))
   )
@@
     (effects (font (size 1.27 1.27)) (justify right bottom))
   )
+  (label "RST" (at 69.85 159.385 0)
+    (effects (font (size 1.27 1.27)) (justify left bottom))
+  )
   (label "SCK" (at 92.075 22.86 0)
     (effects (font (size 1.27 1.27)) (justify left bottom))
   )
   (label "SCK" (at 24.13 157.48 0)
+    (effects (font (size 1.27 1.27)) (justify left bottom))
+  )
+  (label "SDO" (at 69.85 144.145 0)
+    (effects (font (size 1.27 1.27)) (justify left bottom))
+  )
+  (label "SCK" (at 69.85 149.225 0)
+    (effects (font (size 1.27 1.27)) (justify left bottom))
+  )
+  (label "SDI" (at 69.85 154.305 0)
     (effects (font (size 1.27 1.27)) (justify left bottom))
   )
@@
     (pin "1")
   )
+  (symbol (lib_id "Connector:TestPoint") (at 74.93 159.385 270) (unit 1)
+    (in_bom yes) (on_board yes)
+    (property "Reference" "TP404" (id 0) (at 80.01 159.385 90)
+      (effects (font (size 1.27 1.27)) (justify left))
+    )
+    (property "Value" "TestPoint" (id 1) (at 80.645 160.655 90)
+      (effects (font (size 1.27 1.27)) (justify left) hide)
+    )
+    (property "Footprint" "TestPoint:TestPoint_Pad_2.0x2.0mm" (id 2) (at 74.93 164.465 0)
+      (effects (font (size 1.27 1.27)) hide)
+    )
+    (property "Datasheet" "~" (id 3) (at 74.93 164.465 0)
+      (effects (font (size 1.27 1.27)) hide)
+    )
+    (pin "1")
+  )
   (symbol (lib_name "+5V_3") (lib_id "power:+5V") (at 187.96 24.765 0) (unit 1)
     (in_bom yes) (on_board yes)
@@
     (pin "2")
   )
+  (symbol (lib_id "Connector:TestPoint") (at 74.93 144.145 270) (unit 1)
+    (in_bom yes) (on_board yes)
+    (property "Reference" "TP401" (id 0) (at 80.01 144.145 90)
+      (effects (font (size 1.27 1.27)) (justify left))
+    )
+    (property "Value" "TestPoint" (id 1) (at 80.645 145.415 90)
+      (effects (font (size 1.27 1.27)) (justify left) hide)
+    )
+    (property "Footprint" "TestPoint:TestPoint_Pad_2.0x2.0mm" (id 2) (at 74.93 149.225 0)
+      (effects (font (size 1.27 1.27)) hide)
+    )
+    (property "Datasheet" "~" (id 3) (at 74.93 149.225 0)
+      (effects (font (size 1.27 1.27)) hide)
+    )
+    (pin "1")
+  )
   (symbol (lib_id "Device:Crystal") (at 85.09 69.85 180) (unit 1)
     (in_bom yes) (on_board yes)
@@
     (pin "1")
   )
+  (symbol (lib_id "Connector:TestPoint") (at 74.93 154.305 270) (unit 1)
+    (in_bom yes) (on_board yes)
+    (property "Reference" "TP403" (id 0) (at 80.01 154.305 90)
+      (effects (font (size 1.27 1.27)) (justify left))
+    )
+    (property "Value" "TestPoint" (id 1) (at 80.645 155.575 90)
+      (effects (font (size 1.27 1.27)) (justify left) hide)
+    )
+    (property "Footprint" "TestPoint:TestPoint_Pad_2.0x2.0mm" (id 2) (at 74.93 159.385 0)
+      (effects (font (size 1.27 1.27)) hide)
+    )
+    (property "Datasheet" "~" (id 3) (at 74.93 159.385 0)
+      (effects (font (size 1.27 1.27)) hide)
+    )
+    (pin "1")
+  )
   (symbol (lib_name "GND_7") (lib_id "power:GND") (at 27.94 36.83 0) (unit 1)
     (in_bom yes) (on_board yes)
@@
       (effects (font (size 1.27 1.27)) hide)
     )
+    (pin "1")
+  )
+  (symbol (lib_id "Connector:TestPoint") (at 74.93 149.225 270) (unit 1)
+    (in_bom yes) (on_board yes)
+    (property "Reference" "TP402" (id 0) (at 80.01 149.225 90)
+      (effects (font (size 1.27 1.27)) (justify left))
+    )
+    (property "Value" "TestPoint" (id 1) (at 80.645 150.495 90)
+      (effects (font (size 1.27 1.27)) (justify left) hide)
+    )
+    (property "Footprint" "TestPoint:TestPoint_Pad_2.0x2.0mm" (id 2) (at 74.93 154.305 0)
+      (effects (font (size 1.27 1.27)) hide)
+    )
+    (property "Datasheet" "~" (id 3) (at 74.93 154.305 0)
+      (effects (font (size 1.27 1.27)) hide)
+    )

Commit message: Add silkscreen!
Parts:
- removed D401: STAT, LED_SMD:LED_0805_2012Metric, symbol Device:LED
- removed R403: 1K, Resistor_SMD:R_0805_2012Metric, symbol Device:R_Small
- renumbered R404 to R403, R405 to R404
Connections:
- net L_TURN: now reaches U401.10 (PD6)
- net R_TURN: now reaches U401.11 (PD7)
Changed lines of the file:
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@@
-    (stroke (width 0) (type default) (color 0 0 0 0))
-  )
-  (wire (pts (xy 113.665 24.13) (xy 113.665 22.86))
     (stroke (width 0) (type default) (color 0 0 0 0))
   )
@@
     (stroke (width 0) (type default) (color 0 0 0 0))
   )
-  (wire (pts (xy 102.87 22.86) (xy 104.14 22.86))
-    (stroke (width 0) (type default) (color 0 0 0 0))
-  )
   (wire (pts (xy 130.81 32.385) (xy 128.27 32.385))
     (stroke (width 0) (type default) (color 0 0 0 0))
@@
     (stroke (width 0) (type default) (color 0 0 0 0))
   )
+  (wire (pts (xy 80.01 107.315) (xy 57.785 107.315))
+    (stroke (width 0) (type default) (color 0 0 0 0))
+  )
   (wire (pts (xy 80.645 76.835) (xy 80.645 78.74))
     (stroke (width 0) (type default) (color 0 0 0 0))
@@
     (stroke (width 0) (type default) (color 0 0 0 0))
   )
+  (wire (pts (xy 80.01 109.855) (xy 57.785 109.855))
+    (stroke (width 0) (type default) (color 0 0 0 0))
+  )
   (polyline (pts (xy 119.38 13.335) (xy 119.38 60.96))
     (stroke (width 0) (type default) (color 0 0 0 0))
@@
     (stroke (width 0) (type default) (color 0 0 0 0))
   )
-  (wire (pts (xy 92.075 22.86) (xy 97.79 22.86))
-    (stroke (width 0) (type default) (color 0 0 0 0))
-  )
   (wire (pts (xy 88.9 69.85) (xy 89.535 69.85))
     (stroke (width 0) (type default) (color 0 0 0 0))
@@
   )
   (wire (pts (xy 85.09 78.74) (xy 85.09 79.375))
-    (stroke (width 0) (type default) (color 0 0 0 0))
-  )
-  (wire (pts (xy 111.76 22.86) (xy 113.665 22.86))
     (stroke (width 0) (type default) (color 0 0 0 0))
   )
@@
     (effects (font (size 1.27 1.27)) (justify left bottom))
   )
-  (label "SCK" (at 92.075 22.86 0)
-    (effects (font (size 1.27 1.27)) (justify left bottom))
-  )
   (label "SCK" (at 24.13 157.48 0)
     (effects (font (size 1.27 1.27)) (justify left bottom))
@@
   (label "ICSP_RST" (at 24.13 154.94 0)
     (effects (font (size 1.27 1.27)) (justify left bottom))
-  )
-  (label "SCK" (at 79.375 61.595 180)
-    (effects (font (size 1.27 1.27)) (justify right bottom))
   )
   (hierarchical_label "RST" (shape input) (at 82.55 85.725 0)
@@
     (effects (font (size 1.27 1.27)) (justify left))
   )
+  (hierarchical_label "SCK" (shape output) (at 79.375 61.595 0)
+    (effects (font (size 1.27 1.27)) (justify left))
+  )
   (hierarchical_label "DATA_OUT" (shape output) (at 79.375 51.435 0)
     (effects (font (size 1.27 1.27)) (justify left))
   )
+  (hierarchical_label "L_TURN" (shape output) (at 80.01 107.315 0)
+    (effects (font (size 1.27 1.27)) (justify left))
+  )
   (hierarchical_label "LATCH_OUT" (shape output) (at 79.375 53.975 0)
     (effects (font (size 1.27 1.27)) (justify left))
@@
   )
   (hierarchical_label "TXD" (shape output) (at 106.68 94.615 0)
+    (effects (font (size 1.27 1.27)) (justify left))
+  )
+  (hierarchical_label "R_TURN" (shape output) (at 80.01 109.855 0)
     (effects (font (size 1.27 1.27)) (justify left))
   )
@@
     (pin "8")
     (pin "9")
-  )
-  (symbol (lib_id "Device:R_Small") (at 100.33 22.86 270) (unit 1)
-    (in_bom yes) (on_board yes)
-    (property "Reference" "R403" (id 0) (at 100.33 17.78 90))
-    (property "Value" "1K" (id 1) (at 100.33 20.32 90))
-    (property "Footprint" "Resistor_SMD:R_0805_2012Metric" (id 2) (at 100.33 22.86 0)
-      (effects (font (size 1.27 1.27)) hide)
-    )
-    (property "Datasheet" "~" (id 3) (at 100.33 22.86 0)
-      (effects (font (size 1.27 1.27)) hide)
-    )
-    (pin "1")
-    (pin "2")
   )
   (symbol (lib_id "Device:C_Small") (at 27.94 33.02 0) (unit 1)
@@
   (symbol (lib_id "Device:R_Small") (at 130.81 27.305 0) (unit 1)
     (in_bom yes) (on_board yes)
-    (property "Reference" "R404" (id 0) (at 124.46 26.035 0)
+    (property "Reference" "R403" (id 0) (at 124.46 26.035 0)
       (effects (font (size 1.27 1.27)) (justify left))
     )
@@
     (pin "2")
   )
-  (symbol (lib_id "Device:LED") (at 107.95 22.86 180) (unit 1)
-    (in_bom yes) (on_board yes)
-    (property "Reference" "D401" (id 0) (at 107.95 16.51 0))
-    (property "Value" "STAT" (id 1) (at 107.95 19.05 0))
-    (property "Footprint" "LED_SMD:LED_0805_2012Metric" (id 2) (at 107.95 22.86 0)
-      (effects (font (size 1.27 1.27)) hide)
-    )
-    (property "Datasheet" "~" (id 3) (at 107.95 22.86 0)
-      (effects (font (size 1.27 1.27)) hide)
-    )
-    (pin "1")
-    (pin "2")
-  )
   (symbol (lib_name "GND_4") (lib_id "power:GND") (at 146.05 33.655 0) (unit 1)
     (in_bom yes) (on_board yes)
-    (property "Reference" "#PWR0413" (id 0) (at 146.05 40.005 0)
+    (property "Reference" "#PWR0412" (id 0) (at 146.05 40.005 0)
       (effects (font (size 1.27 1.27)) hide)
     )
@@
   (symbol (lib_name "+5V_5") (lib_id "power:+5V") (at 130.81 23.495 0) (unit 1)
     (in_bom yes) (on_board yes)
-    (property "Reference" "#PWR0412" (id 0) (at 130.81 27.305 0)
+    (property "Reference" "#PWR0411" (id 0) (at 130.81 27.305 0)
       (effects (font (size 1.27 1.27)) hide)
     )
@@
   (symbol (lib_name "+5V_3") (lib_id "power:+5V") (at 187.96 24.765 0) (unit 1)
     (in_bom yes) (on_board yes)
-    (property "Reference" "#PWR0415" (id 0) (at 187.96 28.575 0)
+    (property "Reference" "#PWR0414" (id 0) (at 187.96 28.575 0)
       (effects (font (size 1.27 1.27)) hide)
     )
@@
   (symbol (lib_id "Device:R_Small") (at 173.355 31.75 0) (unit 1)
     (in_bom yes) (on_board yes)
-    (property "Reference" "R405" (id 0) (at 166.37 29.845 0)
+    (property "Reference" "R404" (id 0) (at 166.37 29.845 0)
       (effects (font (size 1.27 1.27)) (justify left))
     )
@@
     (pin "2")
   )
-  (symbol (lib_name "GND_10") (lib_id "power:GND") (at 113.665 24.13 0) (unit 1)
-    (in_bom yes) (on_board yes)
-    (property "Reference" "#PWR0411" (id 0) (at 113.665 30.48 0)
-      (effects (font (size 1.27 1.27)) hide)
-    )
-    (property "Value" "GND" (id 1) (at 113.665 27.94 0))
-    (property "Footprint" "" (id 2) (at 113.665 24.13 0)
-      (effects (font (size 1.27 1.27)) hide)
-    )
-    (property "Datasheet" "" (id 3) (at 113.665 24.13 0)
-      (effects (font (size 1.27 1.27)) hide)
-    )
-    (pin "1")
-  )
   (symbol (lib_name "GND_3") (lib_id "power:GND") (at 173.355 36.195 0) (unit 1)
     (in_bom yes) (on_board yes)
-    (property "Reference" "#PWR0414" (id 0) (at 173.355 42.545 0)
-      (effects (font (size 1.27 1.27)) hide)
-    )
+    (property "Reference" "#PWR0413" (id 0) (at 173.355 42.545 0)
+      (effects (font (size 1.27 1.27)) hide)
+    )
