File: Hardware/MegaMouse/mcu.kicad_sch (KiCad schematic)
At the start: 21 parts, among them J401 ICSP, SW401 RESET, SW402 START/MODE, U401 ATmega328P, U402 SN74HC595, Y401 16mHz

Commit message: Carlstrom Review (#2)
Thank you to Professor Carlstrom for reviewing!
Parts:
- renumbered TP406 to TP405
Changed lines of the file:
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@@
   (symbol (lib_id "Connector:TestPoint") (at 172.085 111.125 270) (unit 1)
     (in_bom yes) (on_board yes)
-    (property "Reference" "TP406" (id 0) (at 177.165 111.125 90)
+    (property "Reference" "TP405" (id 0) (at 177.165 111.125 90)
       (effects (font (size 1.27 1.27)) (justify left))
     )

Commit message: Verification 1 (#3)
And thats all we have time for folks.
Parts:
- SW402: LCSC# (none) -> C384611
