File: Hardware/MegaMouse/MegaMouse.kicad_sch (KiCad schematic)
At the start: 15 parts, among them J101 SHIFT_CONN, J102 PROG_CONN, J103 SHIFT_CONN, J104 PROG_CONN

Commit message: Add inital photodiodes
Other:
- sheet IR Sensor renamed FL Sensor
- added sheet FR Sensor (ir_sensor.kicad_sch)
- added sheet FRNT Sensor (ir_sensor.kicad_sch)
- sheet FL Sensor ports: added ENABLE, SENSE; removed none
- sheet MCU ports: added ENABLE, FRNT_IN, LIR_IN, RIR_IN; removed none

Commit message: Add in some more, random junk
Parts:
- removed JP101: BrakeBridge, Jumper:SolderJumper-2_P1.3mm_Bridged_Pad1.0x1.5mm, symbol Jumper:SolderJumper_2_Bridged
Other:
- sheet MCU ports: added BRAKE, L_ENC_A, L_ENC_B, L_MOT_1, L_MOT_2, R_ENC_A, R_ENC_B, R_MOT_1, R_MOT_2; removed SCK
