File: Hardware/MegaMouse/ir_sensor.kicad_sch (KiCad schematic)
At the start: 6 parts

Commit message: Add recomendations from ka2qfx
Parts:
- added R701: 330R, Resistor_SMD:R_0805_2012Metric, symbol Device:R_Small
- H701: renamed from H801; footprint (none) -> MountingHole:MountingHole_3mm
- renumbered R701 to R702, R702 to R703
Connections:
- net +5V: now also R701.1; no longer RV701.1
- new net: R701.2, RV701.1
Changed lines of the file:
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@@
   (junction (at 126.365 97.155) (diameter 0) (color 0 0 0 0)
   )
+  (junction (at 126.365 79.375) (diameter 0) (color 0 0 0 0)
+  )
   (junction (at 126.365 99.695) (diameter 0) (color 0 0 0 0)
-  )
-  (junction (at 126.365 88.9) (diameter 0) (color 0 0 0 0)
   )
   (no_connect (at 115.57 100.965))
@@
     (stroke (width 0) (type default) (color 0 0 0 0))
   )
-  (wire (pts (xy 126.365 88.9) (xy 126.365 90.17))
+  (wire (pts (xy 126.365 79.375) (xy 126.365 90.17))
     (stroke (width 0) (type default) (color 0 0 0 0))
   )
@@
     (stroke (width 0) (type default) (color 0 0 0 0))
   )
+  (wire (pts (xy 115.57 88.9) (xy 115.57 93.345))
+    (stroke (width 0) (type default) (color 0 0 0 0))
+  )
   (wire (pts (xy 126.365 99.695) (xy 126.365 102.87))
     (stroke (width 0) (type default) (color 0 0 0 0))
   )
-  (wire (pts (xy 115.57 88.9) (xy 115.57 93.345))
+  (wire (pts (xy 115.57 79.375) (xy 115.57 83.82))
     (stroke (width 0) (type default) (color 0 0 0 0))
   )
@@
     (stroke (width 0) (type default) (color 0 0 0 0))
   )
-  (wire (pts (xy 126.365 88.9) (xy 115.57 88.9))
+  (wire (pts (xy 126.365 79.375) (xy 115.57 79.375))
     (stroke (width 0) (type default) (color 0 0 0 0))
   )
@@
     (stroke (width 0) (type default) (color 0 0 0 0))
   )
-  (wire (pts (xy 126.365 86.995) (xy 126.365 88.9))
+  (wire (pts (xy 126.365 77.47) (xy 126.365 79.375))
     (stroke (width 0) (type default) (color 0 0 0 0))
   )
@@
   )
   (text "In place of the potentiometer.\nYou can install this resistor\nif an appropriate constant value\nis found."
-    (at 89.535 88.9 0)
+    (at 80.01 87.63 0)
     (effects (font (size 1.27 1.27)) (justify left bottom))
   )
@@
     (pin "1")
   )
+  (symbol (lib_id "Device:R_Small") (at 115.57 86.36 0) (unit 1)
+    (in_bom yes) (on_board yes)
+    (property "Reference" "R701" (id 0) (at 120.015 87.63 0))
+    (property "Value" "330R" (id 1) (at 119.38 85.725 0))
+    (property "Footprint" "Resistor_SMD:R_0805_2012Metric" (id 2) (at 115.57 86.36 0)
+      (effects (font (size 1.27 1.27)) hide)
+    )
+    (property "Datasheet" "~" (id 3) (at 115.57 86.36 0)
+      (effects (font (size 1.27 1.27)) hide)
+    )
+    (pin "1")
+    (pin "2")
+  )
   (symbol (lib_id "Mechanical:MountingHole") (at 15.24 194.31 0) (unit 1)
     (in_bom yes) (on_board yes) (fields_autoplaced)
-    (property "Reference" "H801" (id 0) (at 18.415 193.0399 0)
+    (property "Reference" "H701" (id 0) (at 18.415 193.0399 0)
       (effects (font (size 1.27 1.27)) (justify left))
     )
@@
       (effects (font (size 1.27 1.27)) (justify left))
     )
-    (property "Footprint" "" (id 2) (at 15.24 194.31 0)
+    (property "Footprint" "MountingHole:MountingHole_3mm" (id 2) (at 15.24 194.31 0)
       (effects (font (size 1.27 1.27)) hide)
     )
@@
   (symbol (lib_id "Device:R_Small") (at 146.685 92.71 0) (unit 1)
     (in_bom yes) (on_board yes)
-    (property "Reference" "R702" (id 0) (at 151.13 93.98 0))
+    (property "Reference" "R703" (id 0) (at 151.13 93.98 0))
     (property "Value" "10K" (id 1) (at 150.495 92.075 0))
     (property "Footprint" "Resistor_SMD:R_0805_2012Metric" (id 2) (at 146.685 92.71 0)
@@
     (pin "1")
   )
-  (symbol (lib_id "power:+5V") (at 126.365 86.995 0) (unit 1)
-    (in_bom yes) (on_board yes)
-    (property "Reference" "#PWR0701" (id 0) (at 126.365 90.805 0)
-      (effects (font (size 1.27 1.27)) hide)
-    )
-    (property "Value" "+5V" (id 1) (at 126.365 83.185 0))
-    (property "Footprint" "" (id 2) (at 126.365 86.995 0)
-      (effects (font (size 1.27 1.27)) hide)
-    )
-    (property "Datasheet" "" (id 3) (at 126.365 86.995 0)
+  (symbol (lib_id "power:+5V") (at 126.365 77.47 0) (unit 1)
+    (in_bom yes) (on_board yes)
+    (property "Reference" "#PWR0701" (id 0) (at 126.365 81.28 0)
+      (effects (font (size 1.27 1.27)) hide)
+    )
+    (property "Value" "+5V" (id 1) (at 126.365 73.66 0))
+    (property "Footprint" "" (id 2) (at 126.365 77.47 0)
+      (effects (font (size 1.27 1.27)) hide)
+    )
+    (property "Datasheet" "" (id 3) (at 126.365 77.47 0)
       (effects (font (size 1.27 1.27)) hide)
     )
@@
   (symbol (lib_id "Device:R_Small") (at 126.365 92.71 0) (unit 1)
     (in_bom yes) (on_board yes)
-    (property "Reference" "R701" (id 0) (at 130.81 93.98 0))
+    (property "Reference" "R702" (id 0) (at 130.81 93.98 0))
     (property "Value" "DNP" (id 1) (at 130.175 92.075 0))
     (property "Footprint" "Resistor_SMD:R_0805_2012Metric" (id 2) (at 126.365 92.71 0)
