File: Hardware/MegaMouse/ir_sensor.kicad_sch (KiCad schematic)
At the start: 7 parts

Commit message: Fix ERC
Parts:
- renumbered D701 to D801, D702 to D802, H701 to H801, R701 to R801, R702 to R802, R703 to R803, RV701 to RV801
Changed lines of the file:
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@@
 		(on_board yes)
 		(dnp no)
-		(property "Reference" "#PWR0702"
+		(property "Reference" "#PWR0802"
 			(at 126.365 119.38 0)
 			(effects
@@
 			)
 		)
-		(property "Description" ""
+		(property "Description" "Power symbol creates a global label with name \"GND\" , ground"
 			(at 126.365 113.03 0)
 			(effects
@@
 		(on_board yes)
 		(dnp no)
-		(property "Reference" "R701"
+		(property "Reference" "R801"
 			(at 120.015 87.63 0)
 			(effects
@@
 			)
 		)
-		(property "Description" ""
+		(property "Description" "Resistor, small symbol"
 			(at 115.57 86.36 0)
 			(effects
@@
 		(dnp no)
 		(fields_autoplaced yes)
-		(property "Reference" "H701"
+		(property "Reference" "H801"
 			(at 18.415 193.0399 0)
 			(effects
@@
 			)
 		)
-		(property "Description" ""
+		(property "Description" "Mounting Hole without connection"
 			(at 15.24 194.31 0)
 			(effects
@@
 		(dnp no)
 		(fields_autoplaced yes)
-		(property "Reference" "RV701"
+		(property "Reference" "RV801"
 			(at 113.03 95.8849 0)
 			(effects
@@
 			)
 		)
-		(property "Description" ""
+		(property "Description" "Potentiometer"
 			(at 115.57 97.155 0)
 			(effects
@@
 		(on_board yes)
 		(dnp no)
-		(property "Reference" "D702"
+		(property "Reference" "D802"
 			(at 153.035 107.95 90)
 			(effects
@@
 			)
 		)
-		(property "Description" ""
+		(property "Description" "Light emitting diode"
 			(at 146.685 106.68 0)
 			(effects
@@
 		(on_board yes)
 		(dnp no)
-		(property "Reference" "R703"
+		(property "Reference" "R803"
 			(at 151.13 93.98 0)
 			(effects
@@
 			)
 		)
-		(property "Description" ""
+		(property "Description" "Resistor, small symbol"
 			(at 146.685 92.71 0)
 			(effects
@@
 		(on_board yes)
 		(dnp no)
-		(property "Reference" "D701"
+		(property "Reference" "D801"
 			(at 115.57 106.045 90)
 			(effects
@@
 			)
 		)
-		(property "Description" ""
+		(property "Description" "Photodiode"
 			(at 126.365 107.95 0)
 			(effects
@@
 		(on_board yes)
 		(dnp no)
-		(property "Reference" "#PWR0703"
+		(property "Reference" "#PWR0803"
 			(at 146.685 119.38 0)
 			(effects
@@
 			)
 		)
-		(property "Description" ""
+		(property "Description" "Power symbol creates a global label with name \"GND\" , ground"
 			(at 146.685 113.03 0)
 			(effects
@@
 		(on_board yes)
 		(dnp no)
-		(property "Reference" "#PWR0701"
+		(property "Reference" "#PWR0801"
 			(at 126.365 81.28 0)
 			(effects
@@
 			)
 		)
-		(property "Description" ""
+		(property "Description" "Power symbol creates a global label with name \"+5V\""
 			(at 126.365 77.47 0)
 			(effects
@@
 		(on_board yes)
 		(dnp no)
-		(property "Reference" "R702"
+		(property "Reference" "R802"
 			(at 130.81 93.98 0)
 			(effects
@@
 			)
 		)
-		(property "Description" ""
+		(property "Description" "Resistor, small symbol"
 			(at 126.365 92.71 0)
 			(effects

Commit message: Fix a longstanding bug with tx/rx mismatch (use single footprint now)
Parts:
- renumbered D801 to D701, D802 to D702, H801 to H701, R801 to R701, R802 to R702, R803 to R703, RV801 to RV701
Changed lines of the file:
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@@
 (kicad_sch
-	(version 20231120)
+	(version 20250114)
 	(generator "eeschema")
-	(generator_version "8.0")
+	(generator_version "9.0")
 	(paper "A4")
 	(title_block
@@
 		(comment 4 "Release: ${FULL_REVISION}")
 	)
+	(text "This direction should be correct,\nas the photodiode accepts more light,\nit conducts backwards like this."
+		(exclude_from_sim no)
+		(at 86.36 117.475 0)
+		(effects
+			(font
+				(size 1.27 1.27)
+			)
+			(justify left bottom)
+		)
+	)
+	(text "The IR LED emits light whenever\nENABLE is high.\nIt consumes a similar level of current\nas a red LED."
+		(exclude_from_sim no)
+		(at 150.495 119.38 0)
+		(effects
+			(font
+				(size 1.27 1.27)
+			)
+			(justify left bottom)
+		)
+	)
+	(text "In place of the potentiometer.\nYou can install this resistor\nif an appropriate constant value\nis found."
+		(exclude_from_sim no)
+		(at 80.01 87.63 0)
+		(effects
+			(font
+				(size 1.27 1.27)
+			)
+			(justify left bottom)
+		)
+	)
 	(junction
 		(at 126.365 97.155)
@@
 		)
 	)
-	(text "This direction should be correct,\nas the photodiode accepts more light,\nit conducts backwards like this."
-		(exclude_from_sim no)
-		(at 86.36 117.475 0)
+	(hierarchical_label "SENSE"
+		(shape output)
+		(at 129.54 99.695 0)
 		(effects
 			(font
 				(size 1.27 1.27)
 			)
-			(justify left bottom)
-		)
-	)
-	(text "The IR LED emits light whenever\nENABLE is high.\nIt consumes a similar level of current\nas a red LED."
-		(exclude_from_sim no)
-		(at 150.495 119.38 0)
+			(justify left)
+		)
+	)
+	(hierarchical_label "ENABLE"
+		(shape input)
+		(at 151.765 85.725 0)
 		(effects
 			(font
 				(size 1.27 1.27)
 			)
-			(justify left bottom)
-		)
-	)
-	(text "In place of the potentiometer.\nYou can install this resistor\nif an appropriate constant value\nis found."
-		(exclude_from_sim no)
-		(at 80.01 87.63 0)
-		(effects
-			(font
-				(size 1.27 1.27)
-			)
-			(justify left bottom)
-		)
-	)
-	(hierarchical_label "SENSE"
-		(shape output)
-		(at 129.54 99.695 0)
-		(fields_autoplaced yes)
-		(effects
-			(font
-				(size 1.27 1.27)
-			)
-			(justify left)
-		)
-	)
-	(hierarchical_label "ENABLE"
-		(shape input)
-		(at 151.765 85.725 0)
-		(fields_autoplaced yes)
-		(effects
-			(font
-				(size 1.27 1.27)
-			)
 			(justify left)
 		)
@@
 		(on_board yes)
 		(dnp no)
-		(property "Reference" "#PWR0802"
+		(property "Reference" "#PWR0702"
 			(at 126.365 119.38 0)
 			(effects
@@
 		(on_board yes)
 		(dnp no)
-		(property "Reference" "R801"
+		(property "Reference" "R701"
 			(at 120.015 87.63 0)
 			(effects
@@
 		(dnp no)
 		(fields_autoplaced yes)
-		(property "Reference" "H801"
+		(property "Reference" "H701"
 			(at 18.415 193.0399 0)
 			(effects
@@
 		(dnp no)
 		(fields_autoplaced yes)
-		(property "Reference" "RV801"
+		(property "Reference" "RV701"
 			(at 113.03 95.8849 0)
 			(effects
@@
 		(on_board yes)
 		(dnp no)
-		(property "Reference" "D802"
+		(property "Reference" "D702"
 			(at 153.035 107.95 90)
 			(effects
@@
 		(on_board yes)
 		(dnp no)
-		(property "Reference" "R803"
+		(property "Reference" "R703"
 			(at 151.13 93.98 0)
 			(effects
@@
 		(on_board yes)
 		(dnp no)
-		(property "Reference" "D801"
+		(property "Reference" "D701"
 			(at 115.57 106.045 90)
 			(effects
@@
 		(on_board yes)
 		(dnp no)
-		(property "Reference" "#PWR0803"
+		(property "Reference" "#PWR0703"
 			(at 146.685 119.38 0)
 			(effects
@@
 		(on_board yes)
 		(dnp no)
-		(property "Reference" "#PWR0801"
+		(property "Reference" "#PWR0701"
 			(at 126.365 81.28 0)
 			(effects
@@
 		(on_board yes)
 		(dnp no)
-		(property "Reference" "R802"
+		(property "Reference" "R702"
 			(at 130.81 93.98 0)
 			(effects
