File: Hardware/MegaMouse/motor.kicad_sch (KiCad schematic)
At the start: 4 parts, among them J201 Motor, U201 DRV8871DDA

Commit message: Add recomendations from ka2qfx
Parts:
- added C202: 100nF, Capacitor_SMD:C_0805_2012Metric, symbol Device:C_Small
Connections:
- net +5V: now also C202.2
- net GND: now also C202.1
Changed lines of the file:
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@@
     (comment 4 "Release: ${FULL_REVISION}")
   )
+  (junction (at 153.67 95.885) (diameter 0) (color 0 0 0 0)
+  )
+  (junction (at 149.225 103.505) (diameter 0) (color 0 0 0 0)
+  )
   (junction (at 96.52 85.725) (diameter 0) (color 0 0 0 0)
   )
@@
     (stroke (width 0) (type default) (color 0 0 0 0))
   )
+  (wire (pts (xy 149.225 95.885) (xy 153.67 95.885))
+    (stroke (width 0) (type default) (color 0 0 0 0))
+  )
+  (wire (pts (xy 149.225 103.505) (xy 168.91 103.505))
+    (stroke (width 0) (type default) (color 0 0 0 0))
+  )
   (wire (pts (xy 164.465 100.965) (xy 168.91 100.965))
     (stroke (width 0) (type default) (color 0 0 0 0))
@@
     (stroke (width 0) (type default) (color 0 0 0 0))
   )
-  (wire (pts (xy 147.32 102.235) (xy 147.32 103.505))
+  (wire (pts (xy 139.065 102.235) (xy 139.065 103.505))
     (stroke (width 0) (type default) (color 0 0 0 0))
   )
@@
     (stroke (width 0) (type default) (color 0 0 0 0))
   )
-  (wire (pts (xy 147.32 103.505) (xy 168.91 103.505))
+  (wire (pts (xy 139.065 103.505) (xy 149.225 103.505))
     (stroke (width 0) (type default) (color 0 0 0 0))
   )
@@
   )
   (wire (pts (xy 106.68 104.775) (xy 110.49 104.775))
+    (stroke (width 0) (type default) (color 0 0 0 0))
+  )
+  (wire (pts (xy 149.225 102.235) (xy 149.225 103.505))
+    (stroke (width 0) (type default) (color 0 0 0 0))
+  )
+  (wire (pts (xy 149.225 97.155) (xy 149.225 95.885))
     (stroke (width 0) (type default) (color 0 0 0 0))
   )
@@
     (pin "9")
   )
-  (symbol (lib_id "power:+5V") (at 147.32 102.235 0) (unit 1)
-    (in_bom yes) (on_board yes)
-    (property "Reference" "#PWR0205" (id 0) (at 147.32 106.045 0)
-      (effects (font (size 1.27 1.27)) hide)
-    )
-    (property "Value" "+5V" (id 1) (at 147.32 98.425 0))
-    (property "Footprint" "" (id 2) (at 147.32 102.235 0)
-      (effects (font (size 1.27 1.27)) hide)
-    )
-    (property "Datasheet" "" (id 3) (at 147.32 102.235 0)
+  (symbol (lib_id "power:+5V") (at 139.065 102.235 0) (unit 1)
+    (in_bom yes) (on_board yes)
+    (property "Reference" "#PWR0205" (id 0) (at 139.065 106.045 0)
+      (effects (font (size 1.27 1.27)) hide)
+    )
+    (property "Value" "+5V" (id 1) (at 139.065 98.425 0))
+    (property "Footprint" "" (id 2) (at 139.065 102.235 0)
+      (effects (font (size 1.27 1.27)) hide)
+    )
+    (property "Datasheet" "" (id 3) (at 139.065 102.235 0)
       (effects (font (size 1.27 1.27)) hide)
     )
@@
       (effects (font (size 1.27 1.27)) hide)
     )
+    (pin "1")
+    (pin "2")
+  )
+  (symbol (lib_id "Device:C_Small") (at 149.225 99.695 0) (unit 1)
+    (in_bom yes) (on_board yes)
+    (property "Reference" "C202" (id 0) (at 142.24 95.25 0)
+      (effects (font (size 1.27 1.27)) (justify left))
+    )
+    (property "Value" "100nF" (id 1) (at 142.24 97.79 0)
+      (effects (font (size 1.27 1.27)) (justify left))
+    )
+    (property "Footprint" "Capacitor_SMD:C_0805_2012Metric" (id 2) (at 149.225 99.695 0)
+      (effects (font (size 1.27 1.27)) hide)
+    )
+    (property "Datasheet" "~" (id 3) (at 149.225 99.695 0)
+      (effects (font (size 1.27 1.27)) hide)
+    )
