File: Hardware/MegaMouse/motor.kicad_sch (KiCad schematic)
At the start: 5 parts, among them J201 Motor, U201 DRV8871DDA

Commit message: Confirm encoder
Connections:
- net +5V: now also C202.1, J201.2 (Pin_2); no longer C202.2, J201.5 (Pin_5)
- net GND: now also C202.2, J201.5 (Pin_5); no longer C202.1, J201.2 (Pin_2)
Changed lines of the file:
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@@
     (comment 4 "Release: ${FULL_REVISION}")
   )
-  (junction (at 153.67 95.885) (diameter 0) (color 0 0 0 0)
+  (junction (at 149.225 95.885) (diameter 0) (color 0 0 0 0)
+  )
+  (junction (at 96.52 85.725) (diameter 0) (color 0 0 0 0)
   )
   (junction (at 149.225 103.505) (diameter 0) (color 0 0 0 0)
   )
-  (junction (at 96.52 85.725) (diameter 0) (color 0 0 0 0)
-  )
   (wire (pts (xy 164.465 98.425) (xy 168.91 98.425))
     (stroke (width 0) (type default))
   )
-  (wire (pts (xy 153.67 95.885) (xy 168.91 95.885))
+  (wire (pts (xy 149.225 95.885) (xy 168.91 95.885))
     (stroke (width 0) (type default))
   )
@@
     (stroke (width 0) (type default))
   )
-  (wire (pts (xy 149.225 95.885) (xy 153.67 95.885))
+  (wire (pts (xy 139.065 103.505) (xy 149.225 103.505))
     (stroke (width 0) (type default))
   )
@@
     (stroke (width 0) (type default))
   )
-  (wire (pts (xy 153.67 97.155) (xy 153.67 95.885))
-    (stroke (width 0) (type default))
-  )
   (wire (pts (xy 110.49 113.03) (xy 110.49 111.76))
     (stroke (width 0) (type default))
@@
     (stroke (width 0) (type default))
   )
-  (wire (pts (xy 139.065 102.235) (xy 139.065 103.505))
+  (wire (pts (xy 139.065 94.615) (xy 139.065 95.885))
     (stroke (width 0) (type default))
   )
@@
     (stroke (width 0) (type default))
   )
-  (wire (pts (xy 139.065 103.505) (xy 149.225 103.505))
+  (wire (pts (xy 139.065 95.885) (xy 149.225 95.885))
+    (stroke (width 0) (type default))
+  )
+  (wire (pts (xy 139.065 104.775) (xy 139.065 103.505))
     (stroke (width 0) (type default))
   )
@@
     (stroke (width 0) (type default))
   )
-  (text "GND" (at 174.625 96.52 0)
+  (text "GND" (at 174.625 104.14 0)
     (effects (font (size 0.762 0.762)) (justify left bottom))
   )
@@
     (effects (font (size 0.762 0.762)) (justify left bottom))
   )
-  (text "VCC" (at 174.625 104.14 0)
+  (text "VCC" (at 174.625 96.52 0)
     (effects (font (size 0.762 0.762)) (justify left bottom))
   )
@@
     (effects (font (size 1.27 1.27)) (justify right))
   )
+  (symbol (lib_id "power:GND") (at 139.065 104.775 0) (unit 1)
+    (in_bom yes) (on_board yes) (dnp no)
+    (property "Reference" "#PWR0206" (at 139.065 111.125 0)
+      (effects (font (size 1.27 1.27)) hide)
+    )
+    (property "Value" "GND" (at 139.065 108.585 0)
+      (effects (font (size 1.27 1.27)))
+    )
+    (property "Footprint" "" (at 139.065 104.775 0)
+      (effects (font (size 1.27 1.27)) hide)
+    )
+    (property "Datasheet" "" (at 139.065 104.775 0)
+      (effects (font (size 1.27 1.27)) hide)
+    )
+    (pin "1")
+    (instances
+      (project "MegaMouse"
+        (path "/cb242f39-3922-44b0-8f13-dded6a2d135b/cab2ae08-2794-43d3-b90a-39adfeeefd96"
+          (reference "#PWR0206") (unit 1)
+        )
+        (path "/cb242f39-3922-44b0-8f13-dded6a2d135b/f3134389-3b86-403d-ae8e-c46efd53e738"
+          (reference "#PWR0306") (unit 1)
+        )
+      )
+    )
+  )
   (symbol (lib_id "power:GND") (at 96.52 113.03 0) (unit 1)
     (in_bom yes) (on_board yes) (dnp no)
@@
         (path "/cb242f39-3922-44b0-8f13-dded6a2d135b/f3134389-3b86-403d-ae8e-c46efd53e738"
           (reference "#PWR0301") (unit 1)
-        )
-      )
-    )
-  )
-  (symbol (lib_id "power:GND") (at 153.67 97.155 0) (unit 1)
-    (in_bom yes) (on_board yes) (dnp no)
-    (property "Reference" "#PWR0206" (at 153.67 103.505 0)
-      (effects (font (size 1.27 1.27)) hide)
-    )
-    (property "Value" "GND" (at 153.67 100.965 0)
-      (effects (font (size 1.27 1.27)))
-    )
-    (property "Footprint" "" (at 153.67 97.155 0)
-      (effects (font (size 1.27 1.27)) hide)
-    )
-    (property "Datasheet" "" (at 153.67 97.155 0)
-      (effects (font (size 1.27 1.27)) hide)
-    )
-    (pin "1")
-    (instances
-      (project "MegaMouse"
-        (path "/cb242f39-3922-44b0-8f13-dded6a2d135b/cab2ae08-2794-43d3-b90a-39adfeeefd96"
-          (reference "#PWR0206") (unit 1)
-        )
-        (path "/cb242f39-3922-44b0-8f13-dded6a2d135b/f3134389-3b86-403d-ae8e-c46efd53e738"
-          (reference "#PWR0306") (unit 1)
         )
       )
@@
     )
   )
-  (symbol (lib_id "power:+5V") (at 139.065 102.235 0) (unit 1)
-    (in_bom yes) (on_board yes) (dnp no)
-    (property "Reference" "#PWR0205" (at 139.065 106.045 0)
-      (effects (font (size 1.27 1.27)) hide)
-    )
-    (property "Value" "+5V" (at 139.065 98.425 0)
-      (effects (font (size 1.27 1.27)))
-    )
-    (property "Footprint" "" (at 139.065 102.235 0)
-      (effects (font (size 1.27 1.27)) hide)
-    )
-    (property "Datasheet" "" (at 139.065 102.235 0)
+  (symbol (lib_id "power:+5V") (at 139.065 94.615 0) (unit 1)
+    (in_bom yes) (on_board yes) (dnp no)
+    (property "Reference" "#PWR0205" (at 139.065 98.425 0)
+      (effects (font (size 1.27 1.27)) hide)
+    )
+    (property "Value" "+5V" (at 139.065 90.805 0)
+      (effects (font (size 1.27 1.27)))
+    )
+    (property "Footprint" "" (at 139.065 94.615 0)
+      (effects (font (size 1.27 1.27)) hide)
+    )
+    (property "Datasheet" "" (at 139.065 94.615 0)
       (effects (font (size 1.27 1.27)) hide)
     )
@@
   (symbol (lib_id "Device:C_Small") (at 149.225 99.695 0) (unit 1)
     (in_bom yes) (on_board yes) (dnp no)
-    (property "Reference" "C202" (at 142.24 95.25 0)
+    (property "Reference" "C202" (at 141.605 99.06 0)
       (effects (font (size 1.27 1.27)) (justify left))
     )
-    (property "Value" "100nF" (at 142.24 97.79 0)
+    (property "Value" "100nF" (at 141.605 101.6 0)
       (effects (font (size 1.27 1.27)) (justify left))
     )
