File: Hardware/MegaMouse/motor.kicad_sch (KiCad schematic)
At the start: 3 parts, among them J201 Motor, U201 DRV8871DDA

Commit message: Even more stuff! also bump libs
Parts:
- added R201: 15k, Resistor_SMD:R_0805_2012Metric, symbol Device:R_Small
Connections:
- net +5V: no longer C201.1, U201.5 (VM)
- net GND: now also R201.1
- net IN2: now reaches U201.2 (IN2)
- net IN1: now reaches U201.3 (IN1)
- net at U201.4 (ILIM): now also R201.2
- net EncA: now reaches J201.3 (Pin_3)
- net EncB: now reaches J201.4 (Pin_4)
- new net +BATT: C201.1, U201.5 (VM)
Other:
- note added: "Current protection resistor 15-18k for disable"
- moved on the sheet: C201
Changed lines of the file:
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@@
 (kicad_sch (version 20211123) (generator eeschema)
   (paper "A4")
+  (junction (at 96.52 85.725) (diameter 0) (color 0 0 0 0)
+  )
+  (wire (pts (xy 164.465 98.425) (xy 168.91 98.425))
+    (stroke (width 0) (type default) (color 0 0 0 0))
+  )
   (wire (pts (xy 153.67 95.885) (xy 168.91 95.885))
     (stroke (width 0) (type default) (color 0 0 0 0))
   )
-  (wire (pts (xy 120.015 90.805) (xy 120.015 92.075))
+  (wire (pts (xy 96.52 85.725) (xy 96.52 92.075))
+    (stroke (width 0) (type default) (color 0 0 0 0))
+  )
+  (wire (pts (xy 81.28 99.695) (xy 86.36 99.695))
+    (stroke (width 0) (type default) (color 0 0 0 0))
+  )
+  (wire (pts (xy 126.365 85.725) (xy 96.52 85.725))
+    (stroke (width 0) (type default) (color 0 0 0 0))
+  )
+  (wire (pts (xy 126.365 110.49) (xy 126.365 113.03))
     (stroke (width 0) (type default) (color 0 0 0 0))
   )
@@
     (stroke (width 0) (type default) (color 0 0 0 0))
   )
-  (wire (pts (xy 96.52 90.805) (xy 96.52 92.075))
+  (wire (pts (xy 96.52 83.185) (xy 96.52 85.725))
     (stroke (width 0) (type default) (color 0 0 0 0))
   )
@@
     (stroke (width 0) (type default) (color 0 0 0 0))
   )
-  (wire (pts (xy 96.52 111.76) (xy 96.52 109.855))
+  (wire (pts (xy 126.365 105.41) (xy 126.365 85.725))
+    (stroke (width 0) (type default) (color 0 0 0 0))
+  )
+  (wire (pts (xy 164.465 100.965) (xy 168.91 100.965))
+    (stroke (width 0) (type default) (color 0 0 0 0))
+  )
+  (wire (pts (xy 96.52 113.03) (xy 96.52 109.855))
     (stroke (width 0) (type default) (color 0 0 0 0))
   )
@@
     (stroke (width 0) (type default) (color 0 0 0 0))
   )
+  (wire (pts (xy 110.49 113.03) (xy 110.49 111.76))
+    (stroke (width 0) (type default) (color 0 0 0 0))
+  )
+  (wire (pts (xy 81.28 97.155) (xy 86.36 97.155))
+    (stroke (width 0) (type default) (color 0 0 0 0))
+  )
   (wire (pts (xy 147.32 102.235) (xy 147.32 103.505))
     (stroke (width 0) (type default) (color 0 0 0 0))
   )
+  (wire (pts (xy 110.49 104.775) (xy 110.49 106.68))
+    (stroke (width 0) (type default) (color 0 0 0 0))
+  )
   (wire (pts (xy 147.32 103.505) (xy 168.91 103.505))
     (stroke (width 0) (type default) (color 0 0 0 0))
@@
     (stroke (width 0) (type default) (color 0 0 0 0))
   )
-  (wire (pts (xy 120.015 84.455) (xy 120.015 85.725))
+  (wire (pts (xy 106.68 104.775) (xy 110.49 104.775))
     (stroke (width 0) (type default) (color 0 0 0 0))
   )
@@
   (text "C2" (at 174.625 101.6 0)
     (effects (font (size 0.762 0.762)) (justify left bottom))
+  )
+  (text "Current protection resistor\n15-18k for disable" (at 111.125 113.665 0)
+    (effects (font (size 0.508 0.508)) (justify left bottom))
   )
   (text "M1" (at 174.625 93.98 0)
@@
     (effects (font (size 1.27 1.27)) (justify left bottom))
   )
-  (symbol (lib_id "power:GND") (at 96.52 111.76 0) (unit 1)
-    (in_bom yes) (on_board yes)
-    (property "Reference" "#PWR0202" (id 0) (at 96.52 118.11 0)
-      (effects (font (size 1.27 1.27)) hide)
-    )
-    (property "Value" "GND" (id 1) (at 96.52 115.57 0))
-    (property "Footprint" "" (id 2) (at 96.52 111.76 0)
-      (effects (font (size 1.27 1.27)) hide)
-    )
-    (property "Datasheet" "" (id 3) (at 96.52 111.76 0)
+  (hierarchical_label "IN2" (shape input) (at 81.28 99.695 180)
+    (effects (font (size 1.27 1.27)) (justify right))
+  )
+  (hierarchical_label "EncA" (shape output) (at 164.465 98.425 180)
+    (effects (font (size 1.27 1.27)) (justify right))
+  )
+  (hierarchical_label "IN1" (shape input) (at 81.28 97.155 180)
+    (effects (font (size 1.27 1.27)) (justify right))
+  )
+  (hierarchical_label "EncB" (shape output) (at 164.465 100.965 180)
+    (effects (font (size 1.27 1.27)) (justify right))
+  )
+  (symbol (lib_id "power:GND") (at 96.52 113.03 0) (unit 1)
+    (in_bom yes) (on_board yes)
+    (property "Reference" "#PWR0202" (id 0) (at 96.52 119.38 0)
+      (effects (font (size 1.27 1.27)) hide)
+    )
+    (property "Value" "GND" (id 1) (at 96.52 116.84 0))
+    (property "Footprint" "" (id 2) (at 96.52 113.03 0)
+      (effects (font (size 1.27 1.27)) hide)
+    )
+    (property "Datasheet" "" (id 3) (at 96.52 113.03 0)
+      (effects (font (size 1.27 1.27)) hide)
+    )
+    (pin "1")
+  )
+  (symbol (lib_id "power:+BATT") (at 96.52 83.185 0) (unit 1)
+    (in_bom yes) (on_board yes)
+    (property "Reference" "#PWR0201" (id 0) (at 96.52 86.995 0)
+      (effects (font (size 1.27 1.27)) hide)
+    )
+    (property "Value" "+BATT" (id 1) (at 96.52 79.375 0))
+    (property "Footprint" "" (id 2) (at 96.52 83.185 0)
+      (effects (font (size 1.27 1.27)) hide)
+    )
+    (property "Datasheet" "" (id 3) (at 96.52 83.185 0)
       (effects (font (size 1.27 1.27)) hide)
     )
@@
     (pin "1")
   )
-  (symbol (lib_id "power:+5V") (at 96.52 90.805 0) (unit 1)
-    (in_bom yes) (on_board yes)
-    (property "Reference" "#PWR0201" (id 0) (at 96.52 94.615 0)
-      (effects (font (size 1.27 1.27)) hide)
-    )
-    (property "Value" "+5V" (id 1) (at 96.52 86.995 0))
-    (property "Footprint" "" (id 2) (at 96.52 90.805 0)
-      (effects (font (size 1.27 1.27)) hide)
-    )
-    (property "Datasheet" "" (id 3) (at 96.52 90.805 0)
+  (symbol (lib_id "power:GND") (at 110.49 113.03 0) (unit 1)
+    (in_bom yes) (on_board yes)
+    (property "Reference" "#PWR0203" (id 0) (at 110.49 119.38 0)
+      (effects (font (size 1.27 1.27)) hide)
+    )
+    (property "Value" "GND" (id 1) (at 110.49 116.84 0))
+    (property "Footprint" "" (id 2) (at 110.49 113.03 0)
+      (effects (font (size 1.27 1.27)) hide)
+    )
+    (property "Datasheet" "" (id 3) (at 110.49 113.03 0)
       (effects (font (size 1.27 1.27)) hide)
     )
@@
     (pin "1")
   )
-  (symbol (lib_id "power:+5V") (at 120.015 84.455 0) (unit 1)
-    (in_bom yes) (on_board yes)
-    (property "Reference" "#PWR0203" (id 0) (at 120.015 88.265 0)
-      (effects (font (size 1.27 1.27)) hide)
-    )
-    (property "Value" "+5V" (id 1) (at 120.015 80.645 0))
-    (property "Footprint" "" (id 2) (at 120.015 84.455 0)
-      (effects (font (size 1.27 1.27)) hide)
-    )
-    (property "Datasheet" "" (id 3) (at 120.015 84.455 0)
-      (effects (font (size 1.27 1.27)) hide)
-    )
-    (pin "1")
+  (symbol (lib_id "Device:R_Small") (at 110.49 109.22 180) (unit 1)
+    (in_bom yes) (on_board yes)
+    (property "Reference" "R201" (id 0) (at 114.3 108.585 0))
+    (property "Value" "15k" (id 1) (at 113.665 110.49 0))
+    (property "Footprint" "Resistor_SMD:R_0805_2012Metric" (id 2) (at 110.49 109.22 0)
+      (effects (font (size 1.27 1.27)) hide)
+    )
+    (property "Datasheet" "~" (id 3) (at 110.49 109.22 0)
+      (effects (font (size 1.27 1.27)) hide)
+    )
+    (pin "1")
+    (pin "2")
   )
   (symbol (lib_id "Connector:Conn_01x06_Female") (at 173.99 98.425 0) (unit 1)
@@
     (pin "6")
   )
-  (symbol (lib_id "power:GND") (at 120.015 92.075 0) (unit 1)
-    (in_bom yes) (on_board yes)
-    (property "Reference" "#PWR0204" (id 0) (at 120.015 98.425 0)
-      (effects (font (size 1.27 1.27)) hide)
-    )
-    (property "Value" "GND" (id 1) (at 120.015 95.885 0))
-    (property "Footprint" "" (id 2) (at 120.015 92.075 0)
-      (effects (font (size 1.27 1.27)) hide)
-    )
-    (property "Datasheet" "" (id 3) (at 120.015 92.075 0)
-      (effects (font (size 1.27 1.27)) hide)
-    )
-    (pin "1")
-  )
-  (symbol (lib_id "Device:C_Polarized_Small") (at 120.015 88.265 0) (unit 1)
-    (in_bom yes) (on_board yes)
-    (property "Reference" "C201" (id 0) (at 113.03 86.995 0)
-      (effects (font (size 1.27 1.27)) (justify left))
-    )
-    (property "Value" "10uf" (id 1) (at 113.665 89.535 0)
-      (effects (font (size 1.27 1.27)) (justify left))
-    )
-    (property "Footprint" "Capacitor_SMD:CP_Elec_4x3" (id 2) (at 120.015 88.265 0)
-      (effects (font (size 1.27 1.27)) hide)
-    )
-    (property "Datasheet" "~" (id 3) (at 120.015 88.265 0)
-      (effects (font (size 1.27 1.27)) hide)
-    )
+  (symbol (lib_id "power:GND") (at 126.365 113.03 0) (unit 1)
+    (in_bom yes) (on_board yes)
+    (property "Reference" "#PWR0204" (id 0) (at 126.365 119.38 0)
+      (effects (font (size 1.27 1.27)) hide)
+    )
+    (property "Value" "GND" (id 1) (at 126.365 116.84 0))
+    (property "Footprint" "" (id 2) (at 126.365 113.03 0)
+      (effects (font (size 1.27 1.27)) hide)
+    )
+    (property "Datasheet" "" (id 3) (at 126.365 113.03 0)
+      (effects (font (size 1.27 1.27)) hide)
+    )
+    (pin "1")
+  )
+  (symbol (lib_id "Device:C_Polarized_Small") (at 126.365 107.95 0) (unit 1)
+    (in_bom yes) (on_board yes)
+    (property "Reference" "C201" (id 0) (at 119.38 106.68 0)
+      (effects (font (size 1.27 1.27)) (justify left))
+    )
+    (property "Value" "10uf" (id 1) (at 120.015 109.22 0)
+      (effects (font (size 1.27 1.27)) (justify left))
+    )
+    (property "Footprint" "Capacitor_SMD:CP_Elec_4x3" (id 2) (at 126.365 107.95 0)
+      (effects (font (size 1.27 1.27)) hide)
+    )
+    (property "Datasheet" "~" (id 3) (at 126.365 107.95 0)
+      (effects (font (size 1.27 1.27)) hide)
+    )

Commit message: Bump config
Other:
- company: (none) -> Kitsune Scientific
- title: (none) -> MegaMouse
Changed lines of the file:
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@@
 (kicad_sch (version 20211123) (generator eeschema)
   (paper "A4")
+  (title_block
+    (title "MegaMouse")
+    (date "${ISSUE}")
+    (rev "${REVISION}")
+    (company "Kitsune Scientific")
+    (comment 4 "Release: ${FULL_REVISION}")
+  )
   (junction (at 96.52 85.725) (diameter 0) (color 0 0 0 0)
   )

Commit message: Add more wiring
Connections:
- net M1: now also J201.6 (Pin_6); no longer J201.1 (Pin_1)
- net M2: now also J201.1 (Pin_1); no longer J201.6 (Pin_6)
Changed lines of the file:
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@@
     (effects (font (size 0.508 0.508)) (justify left bottom))
   )
-  (text "M1" (at 174.625 93.98 0)
+  (text "M1" (at 174.625 106.68 0)
     (effects (font (size 0.762 0.762)) (justify left bottom))
   )
@@
     (effects (font (size 0.762 0.762)) (justify left bottom))
   )
-  (text "M2" (at 174.625 106.68 0)
+  (text "M2" (at 174.625 93.98 0)
     (effects (font (size 0.762 0.762)) (justify left bottom))
   )
@@
     (effects (font (size 1.27 1.27)) (justify right bottom))
   )
-  (label "M2" (at 164.465 106.045 0)
-    (effects (font (size 1.27 1.27)) (justify left bottom))
-  )
   (label "M2" (at 111.76 99.695 180)
     (effects (font (size 1.27 1.27)) (justify right bottom))
   )
-  (label "M1" (at 164.465 93.345 0)
+  (label "M2" (at 164.465 93.345 0)
     (effects (font (size 1.27 1.27)) (justify left bottom))
   )
+  (label "M1" (at 164.465 106.045 0)
+    (effects (font (size 1.27 1.27)) (justify left bottom))
+  )

Commit message: Verification 1 (#3)
And thats all we have time for folks.
Parts:
- added C202: 100nF, Capacitor_SMD:C_0805_2012Metric, symbol Device:C_Small
Connections:
- net +5V: now also J201.2 (Pin_2), C202.1; no longer J201.5 (Pin_5)
- net GND: now also J201.5 (Pin_5), C202.2; no longer J201.2 (Pin_2)
