File: Hardware/MegaMouse/power.kicad_sch (KiCad schematic)
At the start: 9 parts, among them SW501 PWR, U501 NCV1117ST50T3G

Commit message: Add BOM
Parts:
- BT501, BT502: LCSC# (none) -> C5290176
- SW501: LCSC# (none) -> C273394
Changed lines of the file:
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@@
+      (effects (font (size 1.27 1.27)) hide)
+    )
+    (property "LCSC#" " C5290176 " (at 98.425 104.14 0)
       (effects (font (size 1.27 1.27)) hide)
     )
@@
       (effects (font (size 1.27 1.27)) hide)
     )
+    (property "LCSC#" "C273394 " (at 111.125 88.265 0)
+      (effects (font (size 1.27 1.27)) hide)
+    )
     (pin "1")
     (pin "2")
@@
       (effects (font (size 1.27 1.27)) hide)
     )
+    (property "LCSC#" " C5290176 " (at 98.425 94.615 0)
+      (effects (font (size 1.27 1.27)) hide)
+    )
