File: Hardware/MegaMouse/power.kicad_sch (KiCad schematic)
At the start: 9 parts, among them SW501 PWR, U501 NCV1117ST50T3G

Commit message: Fix ERC
Other:
- moved on the sheet: BT501, BT502, C501, C502, C503, D501, R501, SW501, U501
