File: Hardware/MegaMouse/upperBoard.kicad_sch (KiCad schematic)
At the start: 32 parts, among them J601 USBC, U601 FT232RL, U602 SN74HC595, U603 STATE

Commit message: Redo segment
Parts:
- removed U603: STATE, Display_7Segment:HDSP-7801, symbol Display_Character:HDSP-7803
- added U604: STATE, KenwoodFox:SM420391N8, symbol KenwoodFox:SM420391N
Connections:
- net GND: now also U604.3 (CA), U604.8 (CA)
- net SEG_A: now also U604.10 (A)
- net SEG_B: now also U604.9 (B)
- net SEG_C: now also U604.7 (C)
- net SEG_D: now also U604.5 (D)
- net SEG_DP: now also U604.6 (DP)
- net SEG_E: now also U604.4 (E)
- net SEG_F: now also U604.2 (F)
- net SEG_G: now also U604.1 (G)
Changed lines of the file:
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@@
-    )
-  )
-  (symbol (lib_id "Display_Character:HDSP-7803") (at 256.54 40.64 0) (unit 1)
-    (in_bom yes) (on_board yes) (dnp no)
-    (property "Reference" "U603" (at 256.54 26.67 0)
-      (effects (font (size 1.27 1.27)))
-    )
-    (property "Value" "STATE" (at 256.54 54.61 0)
-      (effects (font (size 1.27 1.27)))
-    )
-    (property "Footprint" "Display_7Segment:HDSP-7801" (at 256.54 54.61 0)
-      (effects (font (size 1.27 1.27)) hide)
-    )
-    (property "Datasheet" "https://docs.broadcom.com/docs/AV02-2553EN" (at 256.54 40.64 0)
-      (effects (font (size 1.27 1.27)) hide)
-    )
-    (pin "1")
-    (pin "10")
-    (pin "2")
-    (pin "3")
-    (pin "4")
-    (pin "5")
-    (pin "6")
-    (pin "7")
-    (pin "8")
-    (pin "9")
-    (instances
-      (project "MegaMouse"
-        (path "/cb242f39-3922-44b0-8f13-dded6a2d135b/15cf0a12-7ae2-4a92-a2cb-9d52cdb2502c"
-          (reference "U603") (unit 1)
-        )
-      )
     )
   )
@@
         )
       )
+    )
+  )
+  (symbol (lib_id "KenwoodFox:SM420391N") (at 256.54 40.64 0) (unit 1)
+    (in_bom yes) (on_board yes) (dnp no)
+    (property "Reference" "U604" (at 254 26.67 0)
+      (effects (font (size 1.27 1.27)))
+    )
+    (property "Value" "STATE" (at 256.54 54.61 0)
+      (effects (font (size 1.27 1.27)))
+    )
+    (property "Footprint" "KenwoodFox:SM420391N8" (at 256.54 40.64 0)
+      (effects (font (size 1.27 1.27)) hide)
+    )
+    (property "Datasheet" "" (at 256.54 40.64 0)
+      (effects (font (size 1.27 1.27)) hide)
+    )
+    (pin "1")
+    (pin "10")
+    (pin "2")
+    (pin "3")
+    (pin "4")
+    (pin "5")
+    (pin "6")
+    (pin "7")
+    (pin "8")
+    (pin "9")
+    (instances
+      (project "MegaMouse"
+        (path "/cb242f39-3922-44b0-8f13-dded6a2d135b/15cf0a12-7ae2-4a92-a2cb-9d52cdb2502c"
+          (reference "U604") (unit 1)
+        )
+      )

Commit message: Add LCSC part number
Parts:
- U601: LCSC# (none) -> C8690
Changed lines of the file:
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@@
+      (effects (font (size 1.27 1.27)) hide)
+    )
+    (property "LCSC#" "C8690 " (at 125.73 80.01 0)
       (effects (font (size 1.27 1.27)) hide)
     )
